Commit message: 1.fix inertial 2.fix joint name

File: src/description/model/urdf/bot_elf/urdf/bot_elf.urdf (robot description, URDF)
Before this commit: robot bot_elf, 32 links, 31 joints
Links:
- link r_shld_y_link: mass 0 -> 0.397430898254414
Joints:
- removed joint r_knee_y_cod
- added joint r_knee_y_joint: type revolute, parent r_hip_y_link, child r_knee_y_link, origin xyz=0 0 -0.3 rpy=0 0 0, axis 0 1 0, limit lower=0 upper=2.2 effort=150 velocity=20
